Commit message: add opensafehook brushsolarpanel task

File: src/maniskill_myws/assets/safety_hook/mobility.urdf (robot description, URDF)
Before this commit: robot safety_hook, 2 links, 1 joints
Links:
- link base: mass 0.25 -> 0.30; geometry collision box size=0.016 0.020 0.080; collision box size=0.020 0.020 0.150
- link gate: mass 0.05 -> 0.04; geometry collision box size=0.012 0.016 0.130; collision box size=0.014 0.018 0.020
Joints:
- joint gate_hinge: limit lower=0.0 upper=1.22 effort=2.0 velocity=6.0 -> lower=0.0 upper=1.222 effort=5.0 velocity=8.0; origin xyz=0.046875 0.0 0.1328125 rpy=0 0 0 -> xyz=0.030 0.000 0.140 rpy=0 0 0
