Commit message: add new task

File: src/maniskill_myws/assets/globe_valve/base0/mobility.urdf (robot description, URDF)
Before this commit: robot globe_valve, 3 links, 2 joints
Links:
- link handwheel: geometry collision cylinder length=0.02 radius=0.015; collision cylinder length=0.06 radius=0.008
