Commit message: feat:restrict success condition

File: src/maniskill_myws/assets/globe_valve/base0/mobility.urdf (robot description, URDF)
Before this commit: robot globe_valve, 3 links, 2 joints
Links:
- added link handwheel_rim; collision mesh filename=meshes/handwheel_part_0.glb; collision mesh filename=meshes/handwheel_part_1.glb
- link handwheel: geometry collision cylinder length=0.02 radius=0.015; collision cylinder length=0.06 radius=0.008
Joints:
- added joint handwheel_rim_joint: type fixed, parent handwheel, child handwheel_rim, origin xyz=0 0 0 rpy=0 0 0
