Commit message: openSafeDoor2,solarPanelStatic2,turnGlobeValve1

File: src/maniskill_myws/assets/brush/urdf/brush.urdf (robot description, URDF)
Before this commit: robot brush, 1 links, 0 joints
Links:
- link base_link: geometry collision mesh filename=package://brush/meshes/brush2/part_0.glb; collision mesh filename=package://brush/meshes/brush2/part_1.glb

File: src/maniskill_myws/assets/hook2/urdf/hook2.urdf (robot description, URDF)
Before this commit: robot hook2, 2 links, 1 joints
Joints:
- joint joint_bar: limit lower=0 upper=-0.56 effort=0 velocity=0 -> lower=0.09 upper=-0.56 effort=0 velocity=0
