Commit message: hook2 fix, not finished

File: src/maniskill_myws/assets/hook2/urdf/hook2.urdf (robot description, URDF)
Before this commit: robot hook2, 2 links, 1 joints
Links:
- link bar_link: geometry collision mesh filename=package://hook2/meshes/bar_link/part_0.glb; visual mesh filename=package://hook2/meshes/bar_link.glb
- link frame_link: mass 0.072357 -> 100; geometry collision mesh filename=package://hook2/meshes/frame_link/part_0.glb; collision mesh filename=package://hook2/meshes/frame_link/part_1.glb

Commit message: add:TakeSafetyHook1 task

File: src/maniskill_myws/assets/hook2/urdf/hook2.urdf (robot description, URDF)
Before this commit: robot hook2, 2 links, 1 joints
Links:
- link frame_link: mass 100 -> 1.0
Joints:
- joint joint_bar: axis 0 1 0 -> 1 0 0; limit lower=0.09 upper=-0.56 effort=0 velocity=0 -> lower=-0.019 upper=0.0 effort=0 velocity=0; type revolute -> prismatic
